File: BMS Interface/BMS Interface.brd (EAGLE design)
At the start: 69.8 x 82.5 mm, 24 parts

Commit message: UPdating resistor packages to sizes which are
capable of disappating the appropriate amount of power.
Parts:
- R3: device SparkFun-Resistors:0603-RES -> SparkFun-Passives:0805
Routing:
- net N$2: track 4.35 -> 5.12 mm
Other:
- board text added: "Prosthesis BMS Interface V1.1"
- board text removed: "Prosthesis BMS Interface V1.0"
Changed lines of the file:
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@@
 <setting verticaltext="up"/>
 </settings>
-<grid distance="0.05" unitdist="inch" unit="inch" style="lines" multiple="1" display="yes" altdistance="0.005" altunitdist="inch" altunit="inch"/>
+<grid distance="0.0125" unitdist="inch" unit="inch" style="lines" multiple="1" display="yes" altdistance="0.005" altunitdist="inch" altunit="inch"/>
 <layers>
 <layer number="1" name="Top" color="4" fill="1" visible="yes" active="yes"/>
@@
 <text x="46.99" y="2.2225" size="1.016" layer="21" font="vector" ratio="15" rot="R90">-ve</text>
 <text x="24.13" y="70.1675" size="1.778" layer="25" font="vector" ratio="15">Prosthesis BMS
-Interface V1.0</text>
+Interface V1.1</text>
 <text x="12.7" y="11.43" size="1.016" layer="25" font="vector" ratio="15">ANLG OUT (0-5V)</text>
 </plain>
@@
 <element name="U$3" library="SparkFun-Electromechanical" package="RELAY-G5V" value="RELAY-2G5Q" x="40.9575" y="20.0025"/>
 <element name="D3" library="SparkFun-DiscreteSemi" package="SMA-DIODE" value="1n4001" x="32.385" y="20.0025" rot="R90"/>
-<element name="R3" library="SparkFun-Resistors" package="0603-RES" value="1K" x="6.6675" y="78.74" rot="R90"/>
 <element name="FAULT" library="SparkFun-LED" package="LED5MM" value="Red" x="12.065" y="79.0575"/>
 <element name="PWR" library="SparkFun-LED" package="LED5MM" value="GREEN" x="12.065" y="71.755"/>
@@
 <element name="BMS_IO" library="SparkFun-Connectors" package="ATX24_RIGHT_ANGLE" value="ATX24RH" x="10.16" y="39.37" rot="R270"/>
 <element name="U$4" library="prosthesis" package="PROS_LOGO" value="" x="18.0975" y="74.295"/>
+<element name="R3" library="SparkFun-Passives" package="0805" value="1K" x="6.6675" y="78.74" rot="R90"/>
 </elements>
 <signals>
@@
 <contactref element="U$3" pad="5"/>
 <contactref element="U$3" pad="6"/>
-<contactref element="R3" pad="1"/>
 <polygon width="1.4224" layer="1" isolate="0.3048">
 <vertex x="0.635" y="81.915"/>
@@
 <contactref element="BMS_IO" pad="2"/>
 <contactref element="BMS_IO" pad="3"/>
+<contactref element="R3" pad="1"/>
 </signal>
 <signal name="STATE_OF_CHARGE">
@@
 </signal>
 <signal name="N$2">
+<contactref element="FAULT" pad="A"/>
+<wire x1="10.2625" y1="79.59" x2="10.795" y2="79.0575" width="0.3048" layer="1"/>
 <contactref element="R3" pad="2"/>
-<contactref element="FAULT" pad="A"/>
-<wire x1="6.6675" y1="79.59" x2="10.2625" y2="79.59" width="0.3048" layer="1"/>
-<wire x1="10.2625" y1="79.59" x2="10.795" y2="79.0575" width="0.3048" layer="1"/>
+<wire x1="6.6675" y1="79.64" x2="10.2125" y2="79.64" width="0.4064" layer="1"/>
+<wire x1="10.2125" y1="79.64" x2="10.795" y2="79.0575" width="0.4064" layer="1"/>
 </signal>
 </signals>

Commit message: Added capacitors for the three main boards
Parts:
- added C1: 100uF, SparkFun-Capacitors:CPOL-RADIAL-100UF-25V
Connections:
- net 12V_PWR: now also C1.1
- net GND: now also C1.2
Other:
- board text added: "Prosthesis BMS Interface V1.2"
- board text removed: "Prosthesis BMS Interface V1.1"
Changed lines of the file:
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@@
 <text x="46.99" y="2.2225" size="1.016" layer="21" font="vector" ratio="15" rot="R90">-ve</text>
 <text x="24.13" y="70.1675" size="1.778" layer="25" font="vector" ratio="15">Prosthesis BMS
-Interface V1.1</text>
+Interface V1.2</text>
 <text x="12.7" y="11.43" size="1.016" layer="25" font="vector" ratio="15">ANLG OUT (0-5V)</text>
 </plain>
@@
 <element name="U$4" library="prosthesis" package="PROS_LOGO" value="" x="18.0975" y="74.295"/>
 <element name="R3" library="SparkFun-Passives" package="0805" value="1K" x="6.6675" y="78.74" rot="R90"/>
+<element name="C1" library="SparkFun-Capacitors" package="CPOL-RADIAL-100UF-25V" value="100uF" x="51.1175" y="43.4975" rot="R270"/>
 </elements>
 <signals>
@@
 <contactref element="BMS_IO" pad="11"/>
 <contactref element="BMS_IO" pad="12"/>
+<contactref element="C1" pad="2"/>
 </signal>
 <signal name="MULTIPURPOSE_INPUT">
@@
 <contactref element="BMS_IO" pad="3"/>
 <contactref element="R3" pad="1"/>
+<contactref element="C1" pad="1"/>
 </signal>
 <signal name="STATE_OF_CHARGE">
