File: BMS Interface/BMS Interface.sch (EAGLE design)
At the start: 23 parts

Commit message: Added capacitors for the three main boards
Parts:
- added C1: 100uF, SparkFun-Capacitors:CAP_POLPTH1
Connections:
- net 12V_PWR: now also C1.+
- net GND: now also C1.-
Changed lines of the file:
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@@
 <part name="BMS_IO" library="SparkFun-Connectors" deviceset="ATX24" device="RH"/>
 <part name="R3" library="SparkFun-Passives" deviceset="RESISTOR" device="0805-RES" value="1K"/>
+<part name="C1" library="SparkFun-Capacitors" deviceset="CAP_POL" device="PTH1" value="100uF"/>
 </parts>
 <sheets>
@@
 <instance part="BMS_IO" gate="G$1" x="-48.26" y="45.72"/>
 <instance part="R3" gate="G$1" x="-5.08" y="121.92"/>
+<instance part="C1" gate="G$1" x="48.26" y="63.5"/>
 </instances>
 <busses>
@@
 <label x="-30.48" y="58.42" size="1.778" layer="95"/>
 </segment>
+<segment>
+<pinref part="C1" gate="G$1" pin="-"/>
+<wire x1="48.26" y1="58.42" x2="48.26" y2="55.88" width="0.2032" layer="91"/>
+<label x="48.26" y="55.88" size="1.778" layer="95"/>
+</segment>
 </net>
 <net name="MULTIPURPOSE_INPUT" class="0">
@@
 <label x="-68.58" y="25.4" size="1.778" layer="95" rot="R180"/>
 </segment>
-</net>
+<segment>
+<pinref part="C1" gate="G$1" pin="+"/>
+<wire x1="48.26" y1="66.04" x2="48.26" y2="68.58" width="0.2032" layer="91"/>
+<label x="48.26" y="68.58" size="1.778" layer="95"/>
+</segment>
+</net>
